File: MotorcycleBatterIsolator/MotorcycleBatterIsolator.kicad_sch (KiCad schematic)
At the start: 22 parts

Commit message: Finally onto the PCB. SHould just be a route job then sending it off
Parts:
- removed D? (x4): D, symbol Device:D
- removed J? (x2): Conn_01x02_Male, symbol Connector:Conn_01x02_Male
- removed Q? (x2): Q_NMOS_GDS, symbol Device:Q_NMOS_GDS
- removed R? (x2): R, symbol Device:R
- removed R? (x7): 39, R2030:R2030, symbol Device:R
- added BZ1: Buzzer, Buzzer_Beeper:MagneticBuzzer_ProSignal_ABT-410-RC, symbol Device:Buzzer
- added C1, C12, C15, C5, C8: 1uf, Capacitor_SMD:C_0603_1608Metric, symbol Device:C
- added C10, C7: 4.7pF, Capacitor_SMD:C_0603_1608Metric, symbol Device:C
- added C11, C13, C14, C17, C18, C20, C21, C22, C6, C9: 100nf, Capacitor_SMD:C_0603_1608Metric, symbol Device:C
- added C16, C19, C3, C4: 10uf, Capacitor_SMD:C_0603_1608Metric, symbol Device:C
- added C2: 22uF, Capacitor_SMD:C_0805_2012Metric, symbol Device:C
- added D1, D10, D2, D3, D7, D8: D, Diode_SMD:D_SMA, symbol Device:D
- added D11, D6, D9: LED, LED_SMD:LED_0603_1608Metric, symbol Device:LED
- added D12, D13: D_Zener, Diode_SMD:D_MiniMELF, symbol Device:D_Zener
- added J1, J4: Conn_01x04, AndersonPowerPole:APP_2x2, symbol Connector_Generic:Conn_01x04
- added J2: Micro_SD_Card_Det, Connector_Card:microSD_HC_Molex_104031-0811, symbol Connector:Micro_SD_Card_Det
- added J3: Conn_01x06_Female, Connector:Tag-Connect_TC2030-IDC-NL_2x03_P1.27mm_Vertical, symbol Connector:Conn_01x06_Female
- added J5: USB_C_Receptacle_USB2.0, Connector_USB:USB_C_Receptacle_HRO_TYPE-C-31-M-12, symbol Connector:USB_C_Receptacle_USB2.0
- added JP1: Jumper_2_Bridged, Jumper:SolderJumper-2_P1.3mm_Bridged2Bar_Pad1.0x1.5mm, symbol Jumper:Jumper_2_Bridged
- added Q7: 2N7002, Package_TO_SOT_SMD:SOT-23, symbol Transistor_FET:2N7002
- added R1: 2.2M, Resistor_SMD:R_0603_1608Metric, symbol Device:R
- added R10, R11, R15, R27, R28, R30: 10K, Resistor_SMD:R_0603_1608Metric, symbol Device:R
- added R12, R16: DNP, Resistor_SMD:R_0603_1608Metric, symbol Device:R
- added R13, R17, R22, R24: 1K, Resistor_SMD:R_0603_1608Metric, symbol Device:R
- added R14: 0.001, Resistor_SMD:R_2512_6332Metric, symbol Device:R
- added R18, R19: 27, Resistor_SMD:R_0603_1608Metric, symbol Device:R
- added R20, R21, R23, R25: 5k1, Resistor_SMD:R_0603_1608Metric, symbol Device:R
- added R26, R29: 100K, Resistor_SMD:R_0603_1608Metric, symbol Device:R
- added SW1, SW2, SW3, SW4: SW_Push, Button_Switch_SMD:SW_SPST_TL3342, symbol Switch:SW_Push
- added TH1: Thermistor_NTC, Connector_PinHeader_2.54mm:PinHeader_1x02_P2.54mm_Horizontal, symbol Device:Thermistor_NTC
- added U1: MIC5014, Package_SO:SOP-8_3.76x4.96mm_P1.27mm, symbol MIC5014:MIC5014
- added U2, U6: HT75xx-1-SOT89, Package_TO_SOT_SMD:SOT-89-3, symbol Regulator_Linear:HT75xx-1-SOT89
- added U3: W25Q128JVS, Package_SO:SOIC-8_5.23x5.23mm_P1.27mm, symbol Memory_Flash:W25Q128JVS
- added U4: INA219AxD, Package_SO:SOIC-8_3.9x4.9mm_P1.27mm, symbol Analog_ADC:INA219AxD
- added U5: RP2040, MCU_RaspberryPi_and_Boards:RP2040-QFN-56, symbol MCU_RaspberryPi_and_Boards:RP2040
- added Y1: 12M, Crystal:Crystal_SMD_5032-2Pin_5.0x3.2mm, symbol Device:Crystal
- Q2, Q3, Q5, Q6: renamed from Q?; footprint (none) -> Package_TO_SOT_SMD:TO-252-2
- R4: renamed from R?; LCSC (none) -> C175617
Connections:
- net batteryGnd is gone; now on an unnamed net: Q6.3 (S)
- net +12V: now also BZ1.1 (-), C1.1, C16.1, C3.1, D10.1 (K), D2.1 (K), D7.1 (K), SW1.1, U1.1 (V+), U2.2 (VIN), U6.2 (VIN)
- net GND: now also C1.2, C10.2, C11.2, C12.2, C13.2, C14.2, C15.2, C16.2, C17.2, C18.2, C19.2, C2.2, C20.2, C21.2, C22.2, C3.2, C4.2, C5.2, C6.2, C7.2, C8.2, C9.2, D1.2 (A), D12.2 (A), D13.2 (A), D8.2 (A), J1.3 (Pin_3), J1.4 (Pin_4), J2.11 (SHIELD), J2.6 (VSS), J3.5 (Pin_5), J4.3 (Pin_3), J4.4 (Pin_4), J5.A1 (GND), J5.A12 (GND), J5.B1 (GND), J5.B12 (GND), J5.S1 (SHIELD), Q7.2 (S), R1.2, R10.1, R20.1, R21.1, R22.2, R23.1, R24.2, R25.1, R27.1, R30.1, SW2.2, SW3.2, SW4.2, TH1.1, U1.4 (GND), U2.1 (GND), U3.4 (GND), U4.1 (A1), U4.2 (A0), U4.6 (GND), U5.19 (TESTEN), U5.57 (GND), U6.1 (GND); no longer Q2.3 (S), Q3.3 (S)
- net at Q2.1 (G), Q3.1 (G), Q5.1 (G)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: now also D6.2 (A), R12.2, U1.5 (GATE)
- net at Q5.2 (D): now also Q6.2 (D), D7.2 (A), JP1.2 (B), R14.1, U4.7 (IN-); no longer Q2.2 (D)
- net at Q5.3 (S): now also Q2.3 (S), Q3.3 (S), R11.1, R12.1, U1.3 (SOURCE)
- net at R4.1: now also JP1.1 (A)
- net at R4.2: now also D3.1 (K)
- net Motorcycle+: now reaches Q3.2 (D)
- net Motorcycle+: now also Q2.2 (D), D1.1 (K), D2.2 (A), D3.2 (A), J1.1 (Pin_1), J1.2 (Pin_2), R26.1; no longer Q6.2 (D)
- new net: SW4.1, U5.11 (GPIO8)
- new net: SW3.1, U5.12 (GPIO9)
- new net: R17.2, U5.20 (XIN)
- new net: C10.1, U5.21 (XOUT), Y1.2
- new net: J3.4 (Pin_4), U5.24 (SWCLK)
- new net: J3.2 (Pin_2), U5.25 (SWD)
- new net: D11.2 (A), U5.34 (GPIO22)
- new net: D9.2 (A), U5.35 (GPIO23)
- new net: R28.1, TH1.2, U5.40 (GPIO28_ADC2)
- new net: R19.1, U5.46 (USB_DM)
- new net: R18.1, U5.47 (USB_DP)
- new net: U3.7 (IO3), U5.51 (QSPI_SD3)
- new net: U3.6 (CLK), U5.52 (QSPI_SCLK)
- new net: U3.5 (DI(IO0)), U5.53 (QSPI_SD0)
- new net: U3.3 (IO2), U5.54 (QSPI_SD2)
- new net: U3.2 (DO(IO1)), U5.55 (QSPI_SD1)
- new net: R13.2, R16.2, U3.1 (~{CS}), U5.56 (QSPI_SS)
- new net: D11.1 (K), R24.1
- new net: J5.B5 (CC2), R20.2
- new net: J5.A5 (CC1), R21.2
- new net: D9.1 (K), R22.1
- new net: BZ1.2 (+), Q7.3 (D)
- new net: C4.1, C5.1, J2.4 (VDD), U2.3 (VOUT)
- new net: C7.1, R17.1, Y1.1
- new net: D6.1 (K), R11.2
- new net: D10.2 (A), J5.A4 (VBUS), J5.A9 (VBUS), J5.B4 (VBUS), J5.B9 (VBUS)
- new net +1V1: C11.1, C12.1, C9.1, U5.23 (DVDD), U5.45 (VREG_VOUT), U5.50 (DVDD)
- new net +3V3: C13.1, C14.1, C15.1, C17.1, C18.1, C19.1, C20.1, C21.1, C22.1, C6.1, C8.1, J3.1 (Pin_1), R15.2, R16.1, R28.2, U3.8 (VCC), U4.5 (VS), U5.1 (IOVDD), U5.10 (IOVDD), U5.22 (IOVDD), U5.33 (IOVDD), U5.42 (IOVDD), U5.43 (ADC_AVDD), U5.44 (VREG_IN), U5.48 (USB_VDD), U5.49 (IOVDD), U6.3 (VOUT)
- new net BUZZER_CTRL: Q7.1 (G), R10.2, U5.3 (GPIO1)
- new net Battery+: D8.1 (K), J4.1 (Pin_1), J4.2 (Pin_2), R14.2, R29.1, U4.8 (IN+)
- new net BatteryVoltage3v3: D13.1 (K), R29.2, R30.2, U5.39 (GPIO27_ADC1)
- new net DAT0: J2.7 (DAT0), U5.31 (GPIO20)
- new net DAT1: J2.8 (DAT1), U5.30 (GPIO19)
- new net DAT2: J2.1 (DAT2), U5.29 (GPIO18)
- new net DAT3: J2.2 (DAT3/CD), U5.28 (GPIO17)
- new net GATE_CTRL: C2.1, R1.1, SW1.2, U1.2 (INPUT), U5.2 (GPIO0)
- new net MotorcycleVoltage3v3: D12.1 (K), R26.2, R27.2, U5.38 (GPIO26_ADC0)
- new net RST: J3.3 (Pin_3), R15.1, U5.26 (RUN)
- new net SCL: R23.2, U4.4 (SCL), U5.37 (GPIO25)
- new net SDA: R25.2, U4.3 (SDA), U5.36 (GPIO24)
- new net SD_CLK: J2.5 (CLK), U5.18 (GPIO15)
- new net SD_CMD: J2.3 (CMD), U5.27 (GPIO16)
- new net USB_D+: J5.A6 (D+), J5.B6 (D+), R18.2
- new net USB_D-: J5.A7 (D-), J5.B7 (D-), R19.2
- new net ~{USB_BOOT}: R13.1, SW2.1
Other:
- note added: "Ensure Kelvin connection"
- note added: "PGA at /2, full scale 80mV Max current measurement of 50A 1.6mOhm"
- note added: "REMOVE SWITCH IF RP2040 CTRL"
- note added: "SD Card gets its own power supply"
- note added: "Slave address 1000000"
- moved on the sheet: Q2, Q3, Q5, Q6, R4

Commit message: This is the version that got sent off to fab
Parts:
- added H1, H2, H3, H4, H5: H, MountingHole:MountingHole_3.2mm_M3_DIN965_Pad, symbol Mechanical:MountingHole_Pad
- added TP1, TP2, TP3, TP4, TP5, TP6, TP7, TP8: TestPoint, TestPoint:TestPoint_Pad_D1.0mm, symbol Connector:TestPoint
- C1, C12, C15, C5, C8: LCSC Part (none) -> C15849
- C10, C7: LCSC Part (none) -> C1669
- C11, C13, C14, C17, C18, C20, C21, C22, C6, C9: LCSC Part (none) -> C14663
- C16, C19, C3, C4: LCSC Part (none) -> C96446
- C2: LCSC Part (none) -> C45783
- D1, D10, D2, D3, D7, D8: LCSC Part (none) -> C22452
- D11, D6, D9: LCSC Part (none) -> C2286
- D12, D13: LCSC Part (none) -> C8056
- J2: LCSC Part (none) -> C585350
- J5: LCSC Part (none) -> C165948
- Q2, Q3, Q5, Q6: LCSC Part (none) -> C127863
- Q7: LCSC Part (none) -> C8545
- R1: LCSC Part (none) -> C22938
- R10, R11, R15, R27, R28, R30: LCSC (none) -> C25804; LCSC Part (none) -> C25804
- R13, R17, R22, R24: LCSC (none) -> C21190; LCSC Part (none) -> C21190
- R14: LCSC Part (none) -> C312481
- R18, R19: LCSC Part (none) -> C25190
- R20, R21, R23, R25: LCSC Part (none) -> C23186
- R26, R29: LCSC Part (none) -> C25803
- R4: LCSC Part (none) -> C175617
- SW1, SW2, SW3, SW4: LCSC Part (none) -> C318884
- U1: LCSC (none) -> C219121; LCSC Part (none) -> C219121
- U2, U6: LCSC Part (none) -> C14289
- U3: LCSC Part (none) -> C97521
- U4: LCSC Part (none) -> C138706
- U5: LCSC (none) -> C2040; LCSC Part (none) -> C2040
- Y1: LCSC Part (none) -> C90884
Connections:
- net BatteryVoltage3v3: now also U5.40 (GPIO28_ADC2); no longer U5.39 (GPIO27_ADC1)
- net DAT0: now also U5.37 (GPIO25); no longer U5.31 (GPIO20)
- net DAT1: now also U5.36 (GPIO24); no longer U5.30 (GPIO19)
- net DAT2: now also U5.35 (GPIO23); no longer U5.29 (GPIO18)
- net DAT3: now also U5.34 (GPIO22); no longer U5.28 (GPIO17)
- net GND: now also R27.2, H1.1, H2.1, H3.1, H4.1, H5.1; no longer R27.1
- net MotorcycleVoltage3v3: now also R27.1, U5.39 (GPIO27_ADC1); no longer R27.2, U5.38 (GPIO26_ADC0)
- net SCL: now also U5.14 (GPIO11); no longer U5.37 (GPIO25)
- net SDA: now also U5.13 (GPIO10); no longer U5.36 (GPIO24)
- net SD_CLK: now also U5.31 (GPIO20); no longer U5.18 (GPIO15)
- net SD_CMD: now also U5.32 (GPIO21); no longer U5.27 (GPIO16)
- net at U5.15 (GPIO12): now also TP1.1
- net at U5.16 (GPIO13): now also TP2.1
- net at U5.17 (GPIO14): now also TP3.1
- net at D11.2 (A): now also U5.4 (GPIO2); no longer U5.34 (GPIO22)
- net at D9.2 (A): now also U5.5 (GPIO3); no longer U5.35 (GPIO23)
- net Thermistor: now reaches R28.1, TH1.2
- net Thermistor: now also U5.38 (GPIO26_ADC0); no longer U5.40 (GPIO28_ADC2)
- new net: TP4.1, U5.18 (GPIO15)
- new net: TP5.1, U5.27 (GPIO16)
- new net: TP6.1, U5.28 (GPIO17)
- new net: TP7.1, U5.29 (GPIO18)
- new net: TP8.1, U5.30 (GPIO19)
Other:
- moved on the sheet: D11, D9, J5, R22, R23, R24, R25, R27
